File: hardware/midi_controller.sch (KiCad schematic (older format))
At the start: 16 parts, among them J1 DIN5, J2 DIN5, J3 CONN_03, J4 CONN_04, J5 CONN_03, J6 CONN_05, J7 CONN_03, J8 CONN_03, J9 CONN_03, U1 6N137

Commit message: fix analog pins and remove redundant resistor
Parts:
- removed R4: RESISTOR0402, Resistors_Universal:Resistor_SMD+THTuniversal_2512_RM10_HandSoldering_RevA_Date25Jun2010, symbol SparkFun-Resistors:RESISTOR0402
Connections:
- wire segments 108 -> 96
Other:
- moved on the sheet: B1, J1, J2, J3, J4, J5, J6, J7, J8, J9, R1, R2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
